File: hardware/greybadge_pcb/ecp5_25_fpga.kicad_sch (KiCad schematic)
At the start: 19 parts, among them J10 Conn_02x05_Odd_Even, Q1 Q_NMOS_GSD, U13 W25Q128JVSIM, U9 ECP5U_25_CABGA256, X1 SiT2001B

Commit message: feat: rough component placement
Parts:
- removed R22: 10k, Resistor_SMD:R_0805_2012Metric, symbol Device:R
- added RN1C9: 10k, Resistor_SMD:R_0603_1608Metric_Pad0.98x0.95mm_HandSolder, symbol Device:R_Pack04_Split
Connections:
- net GND: now also RN1C9.3 (R3.1)
- net tck: now also RN1C9.6 (R3.2)
- net clkc0_1: now reaches U9.B7 (PT27B/-/PCLKC0_1)
- net clkt0_1: now reaches U9.C7 (PT27A/+/PCLKT0_1)
- net clk0_0: now reaches U9.D7 (PT24B/-/GR_PCLK0_0)
- net clk0_1: now reaches U9.E7 (PT24A/+/GR_PCLK0_1)

Commit message: feat: bga and mcu routing
Parts:
- removed J10: Conn_02x05_Odd_Even, Connector_PinHeader_1.27mm:PinHeader_2x05_P1.27mm_Vertical_SMD, symbol Connector_Generic:Conn_02x05_Odd_Even
- removed RN1C1, RN1C2, RN1C3, RN1C4, RN1C5, RN1C6, RN1C7, RN1C8: 10k, Resistor_SMD:R_0603_1608Metric_Pad0.98x0.95mm_HandSolder, symbol Device:R_Pack04_Split
- added R1, R2, R3, R5, R6, R7, R8, R9: 10K, Resistor_SMD:R_0603_1608Metric_Pad0.98x0.95mm_HandSolder, symbol Device:R
- U13: footprint Package_SO:SOIC-8_5.23x5.23mm_P1.27mm -> Package_SO:SOIC-8_5.3x5.3mm_P1.27mm
Connections:
- net +3.3V: now also R1.2, R2.2, R3.2, R5.2, R6.2, R9.2
- net A5: no longer U9.A15 (PT67B/-)
- net GND: now also R7.2, R8.2
- net cfg_0: now also R8.1
- net cfg_1: now also R9.1
- net cfg_2: now also R7.1
- net creset: now also R6.1
- net sd_clk: now also R1.1
- net sd_cs: now also R5.1
- net sd_io2: now also R3.1
- net sd_io3: now also R2.1
- net B3: now reaches U9.B3 (PT4B/-)
- net B4: now reaches U9.B4 (PT11B/-)
- net B5: now reaches U9.B5 (PT15B/-)
- net B6: now reaches U9.B6 (PT22B/-)
- net B10: now reaches U9.B10 (PT44A/+)
- net B11: now reaches U9.B11 (PT49A/+)
- net B12: now reaches U9.B12 (PT56A/+)
- net B13: now reaches U9.B13 (PT60A/+)
- net B14: now reaches U9.B14 (PT67A/+)
- net B8: now reaches U9.B8 (PT35B/-/PCLKC1_0)
- net B9: now reaches U9.B9 (PT38A/+/GR_PCLK1_0)
- net B15: now reaches U9.B15 (PR2B/-/S0_IN/HS/RDQ8)
- net B16: now reaches U9.B16 (PR2A/+/HS/RDQ8)
- net C15: now reaches U9.C15 (PR5B/-/HS/RDQ8)
- net C16: now reaches U9.C16 (PR5A/+/HS/RDQ8)
- net D16: now reaches U9.D16 (PR8A/+/HS/RDQS8)
- net E15: now reaches U9.E15 (PR8B/-/HS/RDQSN8)
- net E16: now reaches U9.E16 (PR11D/-/RDQ8)
- net tck renamed fpga_tck
- net tdi renamed fpga_tdi
- net tdo renamed fpga_tdo
- net tms renamed fpga_tms
- new net A15: U9.A15 (PT67B/-)

Commit message: Fix annotation
Parts:
- renumbered C53 to C37, C54 to C38, D4 to D2, R28 to R24, R8 to R25, R1 to R26, R9 to R27, R2 to R28, R7 to R29, R3 to R30, R5 to R31, R6 to R32, RN1C9 to RN1C1, TP7 to TP4, U9 to U7, U13 to U8

Commit message: feat: leds
Parts:
- removed RN1C1: 10k, Resistor_SMD:R_0603_1608Metric_Pad0.98x0.95mm_HandSolder, symbol Device:R_Pack04_Split
- added R41: 10K, Resistor_SMD:R_0603_1608Metric_Pad0.98x0.95mm_HandSolder, symbol Device:R
Connections:
- net GND: now also R41.1
- net fpga_tck: now also R41.2
- net C4: now reaches U7.C4 (PT11A/+)
- net C5: now reaches U7.C5 (PT15A/+)
- net C6: now reaches U7.C6 (PT22A/+)
- net D4: now reaches U7.D4 (PT9B/-)
- net D5: now reaches U7.D5 (PT13B/-)
- net D6: now reaches U7.D6 (PT20B/-)
- net C10: now reaches U7.C10 (PT44B/-)
- net C11: now reaches U7.C11 (PT49B/-)
- net C12: now reaches U7.C12 (PT56B/-)
- net C13: now reaches U7.C13 (PT60B/-)
- net CLKT1_0: now reaches U7.C8 (PT35A/+/PCLKT1_0)
- net GR_PCLK_1_1: now reaches U7.C9 (PT38B/-/GR_PCLK1_1)
- net D13: now reaches U7.D13 (PT62A/+)
- net CLKC1_1: now reaches U7.D8 (PT33B/-/PCLKC1_1)
- net E13: now reaches U7.E13 (PT62B/-)
- net CLKT1_1: now reaches U7.E8 (PT33A/+/PCLKT1_1)
- net C3: now reaches U7.C3 (PL2C/+/LDQ8)
- net D3: now reaches U7.D3 (PL2D/-/LDQ8)
- net C14: now reaches U7.C14 (PR2C/+/RDQ8)
- net D14: now reaches U7.D14 (PR2D/-/RDQ8)
- net E14: now reaches U7.E14 (PR5C/+/RDQ8)
Other:
- moved on the sheet: U7B

Commit message: feat: routing cleanupish, power splitting and drc
Connections:
- net +1V1 renamed +F1V1
- net +2V5 renamed +F2V5
- net +3.3V renamed +F3V3

Commit message: Clean up PCB
Parts:
- C36: renamed from C37; footprint Capacitor_SMD:C_0805_2012Metric -> Capacitor_SMD:C_0402_1005Metric
- C37: renamed from C38; footprint Capacitor_SMD:C_0805_2012Metric -> Capacitor_SMD:C_0402_1005Metric
- renumbered D2 to D10, R24 to R32, R41 to R33, R25 to R34, R26 to R35, R27 to R36, R28 to R37, R29 to R38, R30 to R39, R31 to R40, R32 to R41, TP4 to TP6
