File: hardware/greybadge_pcb/ecp5_25_fpga.kicad_sch (KiCad schematic)
At the start: 17 parts, among them Q1 Q_NMOS_GSD, U7 ECP5U_25_CABGA256, U8 W25Q128JVSIM, X1 SiT2001B

Commit message: Add onboard oled (incomplete)
Parts:
- renumbered C41 to C42, C42 to C43, Q1 to Q2, R35 to R38, R36 to R39, R37 to R40, R38 to R41, R39 to R42, R40 to R43, R41 to R44, R42 to R45, R43 to R46, R44 to R47, U7 to U8, U8 to U9

Commit message: Fix prev commit
Parts:
- renumbered R38 to R37, R39 to R38, R40 to R39, R41 to R40, R42 to R41, R43 to R42, R44 to R43, R45 to R44, R46 to R45, R47 to R46

Commit message: feat: stuff
Connections:
- net D12: now reaches U8.D12 (PT58A/+)
